Commit message: some changes to grasp target

File: urdf/robotiq.urdf (robot description, URDF)
Before this commit: robot fanuc_m_20id, 13 links, 12 joints
Joints:
- joint finger_1_joint_1: limit lower=0 upper=1.2211 effort=100 velocity=10 -> lower=0 upper=1.2211 velocity=10
- joint finger_1_joint_2: limit lower=0 upper=1.350 effort=100 velocity=100 -> lower=0 upper=1.350 velocity=100
- joint finger_1_joint_3: limit lower=-0.900 upper=0.75 effort=100 velocity=100 -> lower=-0.900 upper=0.75 velocity=100
- joint finger_2_joint_1: limit lower=0 upper=1.2211 effort=100 velocity=100 -> lower=0 upper=1.2211 velocity=100
- joint finger_2_joint_2: limit lower=0 upper=1.350 effort=100 velocity=100 -> lower=0 upper=1.350 velocity=100
- joint finger_2_joint_3: limit lower=-0.900 upper=0.75 effort=100 velocity=100 -> lower=-0.900 upper=0.75 velocity=100
- joint finger_middle_joint_1: limit lower=0 upper=1.2211 effort=100 velocity=100 -> lower=0 upper=1.2211 velocity=100
- joint finger_middle_joint_2: limit lower=0 upper=1.350 effort=100 velocity=100 -> lower=0 upper=1.350 velocity=100
- joint finger_middle_joint_3: limit lower=-0.900 upper=0.75 effort=100 velocity=100 -> lower=-0.900 upper=0.75 velocity=100
- joint palm_finger_1_joint: limit lower=-0.16 upper=0.25 effort=100 velocity=100 -> lower=-0.16 upper=0.25 velocity=100
- joint palm_finger_2_joint: limit lower=-0.16 upper=0.25 effort=100 velocity=100 -> lower=-0.16 upper=0.25 velocity=100

Commit message: new changes

File: urdf/robotiq.urdf (robot description, URDF)
Before this commit: robot robotiq, 13 links, 12 joints
Links:
- link finger_1_link_3: geometry collision mesh filename=urdf/meshes/collision/link3.stl; visual mesh filename=meshes/visual/link_3.dae
