Commit message: starting changes

File: urdf/block.urdf (robot description, URDF)
Before this commit: robot block_2, 1 links, 0 joints
Links:
- link block_2_base_link: geometry collision box size=0.20 0.2 0.04; visual box size=0.20 0.2 0.04

Commit message: new changes

File: urdf/block.urdf (robot description, URDF)
Before this commit: robot block_2, 1 links, 0 joints
Links:
- link block_2_base_link: geometry collision box size=0.20 0.2 0.02; visual box size=0.20 0.2 0.02

File: urdf/robotiq.urdf (robot description, URDF)
Before this commit: robot fanuc_m_20id, 13 links, 12 joints
Joints:
- joint finger_1_joint_1: limit lower=0 upper=1.2211 effort=100 velocity=100 -> lower=0 upper=1.2211 effort=100 velocity=10

Commit message: contact is improved

File: urdf/block.urdf (robot description, URDF)
Before this commit: robot block_2, 1 links, 0 joints
Links:
- link block_2_base_link: geometry collision box size=0.20 0.2 0.04; visual box size=0.20 0.2 0.04

File: urdf/robotiq.urdf (robot description, URDF)
Before this commit: robot fanuc_m_20id, 13 links, 12 joints
Joints:
- joint palm_finger_1_joint: limit lower=-0.16 upper=0.25 velocity=100 -> (none)
- joint palm_finger_2_joint: limit lower=-0.16 upper=0.25 velocity=100 -> (none)

Commit message: stl file improved and finger controller got better

File: urdf/block.urdf (robot description, URDF)
Before this commit: robot block_2, 1 links, 0 joints
Links:
- removed link block_2_base_link
- added link block_link; collision mesh filename=urdf/target.stl scale=1 1 1; visual mesh filename=urdf/target.stl scale=1 1 1

File: urdf/robotiq.urdf (robot description, URDF)
Before this commit: robot fanuc_m_20id, 13 links, 12 joints
Links:
- link finger_1_link_3: geometry collision mesh filename=meshes/collision/link3.stl; visual mesh filename=meshes/visual/link_3.dae
- link finger_2_link_3: geometry collision mesh filename=meshes/collision/link3.stl; visual mesh filename=meshes/visual/link_3.dae
- link finger_middle_link_3: geometry collision mesh filename=meshes/collision/link3.stl; visual mesh filename=meshes/visual/link_3.dae

Commit message: ready for curruculum learning

File: urdf/block.urdf (robot description, URDF)
Before this commit: robot block, 1 links, 0 joints
Links:
- link block_link: mass None -> 1

Commit message: some test for closing added

File: urdf/block.urdf (robot description, URDF)
Before this commit: robot block, 1 links, 0 joints
Links:
- link block_link: mass 1 -> None

File: urdf/robotiq.urdf (robot description, URDF)
Before this commit: robot robotiq, 13 links, 12 joints
Links:
- link finger_1_link_3: geometry collision mesh filename=urdf/meshes/collision/link_3.STL; visual mesh filename=meshes/visual/link_3.dae
- link finger_2_link_3: geometry collision mesh filename=meshes/collision/link_3.STL; visual mesh filename=meshes/visual/link_3.dae
- link finger_middle_link_3: geometry collision mesh filename=meshes/collision/link_3.STL; visual mesh filename=meshes/visual/link_3.dae
Joints:
- joint finger_1_joint_1: limit lower=0 upper=1.2211 velocity=10 -> lower=0 upper=1.1694 velocity=100
- joint finger_1_joint_2: limit lower=0 upper=1.350 velocity=100 -> lower=0 upper=1.5708 velocity=100
- joint finger_1_joint_3: limit lower=-0.900 upper=0.75 velocity=100 -> lower=-0.9599 upper=0.7505 velocity=100
- joint finger_2_joint_1: limit lower=0 upper=1.2211 velocity=100 -> lower=0 upper=1.1694 velocity=100
- joint finger_2_joint_2: limit lower=0 upper=1.350 velocity=100 -> lower=0 upper=1.5708 velocity=100
- joint finger_2_joint_3: limit lower=-0.900 upper=0.75 velocity=100 -> lower=-0.9599 upper=0.7505 velocity=100
- joint finger_middle_joint_1: limit lower=0 upper=1.2211 velocity=100 -> lower=0 upper=1.1694 velocity=100
- joint finger_middle_joint_2: limit lower=0 upper=1.350 velocity=100 -> lower=0 upper=1.5708 velocity=100
- joint finger_middle_joint_3: limit lower=-0.900 upper=0.75 velocity=100 -> lower=-0.9599 upper=0.7505 velocity=100

Commit message: Clean up code and add plots for 500 random episodes

File: urdf/block.urdf (robot description, URDF)
Before this commit: robot block, 1 links, 0 joints
Links:
- link block_link: mass None -> 1.0
